Commit message: run ok

File: resources/robots/biped/meshes/sa01_rl.urdf (robot description, URDF)
Before this commit: robot sa01, 15 links, 14 joints
Links:
- link LINK_ANKLE_PITCH_L: geometry visual mesh filename=../meshes/LINK_ANKLE_PITCH_L.STL
- link LINK_ANKLE_PITCH_R: geometry visual mesh filename=../meshes/LINK_ANKLE_PITCH_R.STL
- link LINK_HIP_ROLL_L: geometry visual mesh filename=../meshes/LINK_HIP_ROLL_L.STL
- link LINK_HIP_ROLL_R: geometry visual mesh filename=../meshes/LINK_HIP_ROLL_R.STL
- link LINK_HIP_YAW_L: geometry visual mesh filename=../meshes/LINK_HIP_YAW_L.STL
- link LINK_HIP_YAW_R: geometry visual mesh filename=../meshes/LINK_HIP_YAW_R.STL
- link LINK_KNEE_PITCH_L: geometry visual mesh filename=../meshes/LINK_KNEE_PITCH_L.STL
- link LINK_KNEE_PITCH_R: geometry visual mesh filename=../meshes/LINK_KNEE_PITCH_R.STL
