Commit message: adjust urdf

File: resources/robots/biped/urdf/sa01_rl.urdf (robot description, URDF)
Before this commit: robot sa01, 15 links, 14 joints
Links:
- link LINK_HIP_PITCH_L: geometry collision sphere radius=0.02; visual mesh filename=../meshes/LINK_HIP_PITCH_L.STL
- link LINK_HIP_PITCH_R: geometry visual mesh filename=../meshes/LINK_HIP_PITCH_R.STL
- link LINK_KNEE_PITCH_L: geometry collision mesh filename=../meshes/LINK_KNEE_PITCH_L.STL; visual mesh filename=../meshes/LINK_KNEE_PITCH_L.STL
- link LINK_KNEE_PITCH_R: geometry collision mesh filename=../meshes/LINK_KNEE_PITCH_R.STL; visual mesh filename=../meshes/LINK_KNEE_PITCH_R.STL
